File: slave/hardware/kicad/digital_inputs.kicad_sch (KiCad schematic)
At the start: 44 parts, among them IC10 ESDALC6V1W5_SPLIT, IC11 ESDALC6V1W5_SPLIT

Commit message: feat(HW): continue PCB layout and routing updates
Connections:
- net at R53.1, R56.2: now also IC10.3; no longer IC10.5
- net at R52.1, R55.2: now also IC10.5; no longer IC10.3
- net at R43.1, R46.2: now also IC10.1; no longer IC10.4
- net at R42.1, R45.2: now also IC10.4; no longer IC10.1
